File: ActiveSplitterCoverPCB/ActiveSplitterCover.kicad_sch (KiCad schematic)
At the start: 5 parts, among them J10 Conn_01x01_Pin, J6 Conn_01x28_Pin, J7 Conn_01x28_Pin, J8 Conn_01x12_Pin, J9 Conn_01x12_Pin

Commit message: update size of cover PCB
Parts:
- J6, J7: value Conn_01x28_Pin -> Conn_01x24_Pin; footprint Connector_PinHeader_2.54mm:PinHeader_1x28_P2.54mm_Vertical -> Connector_PinHeader_2.54mm:PinHeader_1x24_P2.54mm_Vertical; symbol Connector:Conn_01x28_Pin -> Connector:Conn_01x24_Pin
Connections:
- net GND: no longer J6.25 (Pin_25), J6.26 (Pin_26), J6.27 (Pin_27), J6.28 (Pin_28), J7.25 (Pin_25), J7.26 (Pin_26), J7.27 (Pin_27), J7.28 (Pin_28)
Changed lines of the file:
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@@
   (junction (at 140.97 90.17) (diameter 0) (color 0 0 0 0)
   )
-  (junction (at 160.02 74.93) (diameter 0) (color 0 0 0 0)
-  )
   (junction (at 185.42 92.71) (diameter 0) (color 0 0 0 0)
   )
-  (junction (at 185.42 135.89) (diameter 0) (color 0 0 0 0)
-  )
   (junction (at 160.02 115.57) (diameter 0) (color 0 0 0 0)
   )
@@
   (junction (at 185.42 115.57) (diameter 0) (color 0 0 0 0)
   )
-  (junction (at 185.42 138.43) (diameter 0) (color 0 0 0 0)
-  )
   (junction (at 160.02 130.81) (diameter 0) (color 0 0 0 0)
   )
@@
   (junction (at 123.19 95.25) (diameter 0) (color 0 0 0 0)
   )
-  (junction (at 160.02 135.89) (diameter 0) (color 0 0 0 0)
-  )
   (junction (at 185.42 105.41) (diameter 0) (color 0 0 0 0)
   )
@@
   (junction (at 160.02 133.35) (diameter 0) (color 0 0 0 0)
   )
-  (junction (at 160.02 72.39) (diameter 0) (color 0 0 0 0)
-  )
   (junction (at 185.42 128.27) (diameter 0) (color 0 0 0 0)
   )
@@
   (junction (at 160.02 90.17) (diameter 0) (color 0 0 0 0)
   )
-  (junction (at 160.02 138.43) (diameter 0) (color 0 0 0 0)
-  )
   (junction (at 123.19 97.79) (diameter 0) (color 0 0 0 0)
   )
@@
   (junction (at 185.42 120.65) (diameter 0) (color 0 0 0 0)
   )
-  (junction (at 185.42 72.39) (diameter 0) (color 0 0 0 0)
-  )
   (junction (at 185.42 97.79) (diameter 0) (color 0 0 0 0)
   )
@@
   (junction (at 160.02 95.25) (diameter 0) (color 0 0 0 0)
   )
-  (junction (at 185.42 74.93) (diameter 0) (color 0 0 0 0)
-  )
   (junction (at 185.42 125.73) (diameter 0) (color 0 0 0 0)
   )
@@
     (stroke (width 0) (type default))
   )
-  (wire (pts (xy 160.02 135.89) (xy 160.02 138.43))
+  (wire (pts (xy 160.02 133.35) (xy 160.02 134.62))
     (stroke (width 0) (type default))
   )
@@
     (stroke (width 0) (type default))
   )
-  (wire (pts (xy 185.42 138.43) (xy 185.42 139.7))
-    (stroke (width 0) (type default))
-  )
   (wire (pts (xy 160.02 113.03) (xy 160.02 115.57))
     (stroke (width 0) (type default))
   )
-  (wire (pts (xy 185.42 135.89) (xy 185.42 138.43))
+  (wire (pts (xy 185.42 133.35) (xy 185.42 135.128))
     (stroke (width 0) (type default))
   )
@@
     (stroke (width 0) (type default))
   )
-  (wire (pts (xy 160.02 72.39) (xy 160.02 74.93))
-    (stroke (width 0) (type default))
-  )
   (wire (pts (xy 123.19 72.39) (xy 123.19 74.93))
     (stroke (width 0) (type default))
@@
     (stroke (width 0) (type default))
   )
-  (wire (pts (xy 160.02 133.35) (xy 160.02 135.89))
-    (stroke (width 0) (type default))
-  )
-  (wire (pts (xy 160.02 138.43) (xy 160.02 139.7))
-    (stroke (width 0) (type default))
-  )
   (wire (pts (xy 160.02 85.09) (xy 160.02 87.63))
     (stroke (width 0) (type default))
@@
     (stroke (width 0) (type default))
   )
-  (wire (pts (xy 185.42 69.85) (xy 185.42 72.39))
-    (stroke (width 0) (type default))
-  )
-  (wire (pts (xy 185.42 72.39) (xy 185.42 74.93))
-    (stroke (width 0) (type default))
-  )
   (wire (pts (xy 160.02 90.17) (xy 160.02 92.71))
     (stroke (width 0) (type default))
@@
     (stroke (width 0) (type default))
   )
-  (wire (pts (xy 160.02 69.85) (xy 160.02 72.39))
-    (stroke (width 0) (type default))
-  )
   (wire (pts (xy 185.42 120.65) (xy 185.42 123.19))
     (stroke (width 0) (type default))
@@
   )
   (wire (pts (xy 140.97 72.39) (xy 140.97 74.93))
-    (stroke (width 0) (type default))
-  )
-  (wire (pts (xy 185.42 133.35) (xy 185.42 135.89))
     (stroke (width 0) (type default))
   )
@@
     )
   )
-  (symbol (lib_id "Connector:Conn_01x28_Pin") (at 180.34 102.87 0) (unit 1)
+  (symbol (lib_id "Connector:Conn_01x24_Pin") (at 180.34 102.87 0) (unit 1)
     (in_bom yes) (on_board yes) (dnp no) (fields_autoplaced)
-    (property "Reference" "J7" (at 180.975 65.6295 0)
-      (effects (font (size 1.27 1.27)))
-    )
-    (property "Value" "Conn_01x28_Pin" (at 180.975 68.0537 0)
-      (effects (font (size 1.27 1.27)))
-    )
-    (property "Footprint" "Connector_PinHeader_2.54mm:PinHeader_1x28_P2.54mm_Vertical" (at 180.34 102.87 0)
+    (property "Reference" "J7" (at 180.975 70.7095 0)
+      (effects (font (size 1.27 1.27)))
+    )
+    (property "Value" "Conn_01x24_Pin" (at 180.975 73.1337 0)
+      (effects (font (size 1.27 1.27)))
+    )
+    (property "Footprint" "Connector_PinHeader_2.54mm:PinHeader_1x24_P2.54mm_Vertical" (at 180.34 102.87 0)
       (effects (font (size 1.27 1.27)) hide)
     )
@@
     (pin "16")
     (pin "2")
-    (pin "28")
     (pin "3")
     (pin "5")
@@
     (pin "22")
     (pin "6")
-    (pin "27")
     (pin "9")
     (pin "18")
@@
     (pin "19")
     (pin "13")
-    (pin "26")
     (pin "15")
     (pin "23")
-    (pin "25")
     (pin "1")
     (pin "12")
@@
     )
   )
-  (symbol (lib_id "Connector:Conn_01x28_Pin") (at 154.94 102.87 0) (unit 1)
+  (symbol (lib_id "Connector:Conn_01x24_Pin") (at 154.94 102.87 0) (unit 1)
     (in_bom yes) (on_board yes) (dnp no) (fields_autoplaced)
-    (property "Reference" "J6" (at 155.575 65.6295 0)
-      (effects (font (size 1.27 1.27)))
-    )
-    (property "Value" "Conn_01x28_Pin" (at 155.575 68.0537 0)
-      (effects (font (size 1.27 1.27)))
-    )
-    (property "Footprint" "Connector_PinHeader_2.54mm:PinHeader_1x28_P2.54mm_Vertical" (at 154.94 102.87 0)
+    (property "Reference" "J6" (at 155.575 70.7095 0)
+      (effects (font (size 1.27 1.27)))
+    )
+    (property "Value" "Conn_01x24_Pin" (at 155.575 73.1337 0)
+      (effects (font (size 1.27 1.27)))
+    )
+    (property "Footprint" "Connector_PinHeader_2.54mm:PinHeader_1x24_P2.54mm_Vertical" (at 154.94 102.87 0)
       (effects (font (size 1.27 1.27)) hide)
     )
@@
     (pin "2")
     (pin "24")
-    (pin "25")
-    (pin "28")
     (pin "16")
     (pin "12")
@@
     (pin "22")
     (pin "23")
-    (pin "26")
     (pin "20")
-    (pin "27")
     (pin "17")
     (instances
@@
     )
   )
-  (symbol (lib_id "ActiveSplitter-eagle-import:GND") (at 185.42 142.24 0) (unit 1)
+  (symbol (lib_id "ActiveSplitter-eagle-import:GND") (at 185.42 137.668 0) (unit 1)
     (in_bom yes) (on_board yes) (dnp no)
-    (property "Reference" "#GND04" (at 185.42 142.24 0)
-      (effects (font (size 1.27 1.27)) hide)
-    )
-    (property "Value" "GND" (at 182.88 144.78 0)
+    (property "Reference" "#GND04" (at 185.42 137.668 0)
+      (effects (font (size 1.27 1.27)) hide)
+    )
+    (property "Value" "GND" (at 182.88 140.208 0)
       (effects (font (size 1.4986 1.4986)) (justify left bottom))
     )
-    (property "Footprint" "" (at 185.42 142.24 0)
-      (effects (font (size 1.27 1.27)) hide)
-    )
-    (property "Datasheet" "" (at 185.42 142.24 0)
+    (property "Footprint" "" (at 185.42 137.668 0)
+      (effects (font (size 1.27 1.27)) hide)
+    )
+    (property "Datasheet" "" (at 185.42 137.668 0)
       (effects (font (size 1.27 1.27)) hide)
     )
@@
     )
   )
-  (symbol (lib_id "ActiveSplitter-eagle-import:GND") (at 160.02 142.24 0) (unit 1)
+  (symbol (lib_id "ActiveSplitter-eagle-import:GND") (at 160.02 137.16 0) (unit 1)
     (in_bom yes) (on_board yes) (dnp no)
-    (property "Reference" "#GND03" (at 160.02 142.24 0)
-      (effects (font (size 1.27 1.27)) hide)
-    )
-    (property "Value" "GND" (at 157.48 144.78 0)
+    (property "Reference" "#GND03" (at 160.02 137.16 0)
+      (effects (font (size 1.27 1.27)) hide)
+    )
+    (property "Value" "GND" (at 157.48 139.7 0)
       (effects (font (size 1.4986 1.4986)) (justify left bottom))
     )
-    (property "Footprint" "" (at 160.02 142.24 0)
-      (effects (font (size 1.27 1.27)) hide)
-    )
-    (property "Datasheet" "" (at 160.02 142.24 0)
-      (effects (font (size 1.27 1.27)) hide)
-    )
+    (property "Footprint" "" (at 160.02 137.16 0)
+      (effects (font (size 1.27 1.27)) hide)
+    )
+    (property "Datasheet" "" (at 160.02 137.16 0)
+      (effects (font (size 1.27 1.27)) hide)
+    )
